File: pcb/U3A.kicad_pcb (KiCad board)
At the start: 2 copper layers, 34.5 x 26.4 mm, 38 parts, among them J1 Conn_01x03_Pin, J2 Conn_01x07_Pin, J3 USB_C, J4 Conn_01x08_Pin, Q1 AO3401A, SW1 SW_DIP_x02, U1 LD1117S33TR, U2 FT232RL

Commit message: Update to KiCAD 9
Connections:
- net CTS renamed /CTS
- net RTS renamed /RTS
- net RXD renamed /RXD
- net TXD renamed /TXD
